Commit message: Orgnize urdf files

File: src/robot_description/models/myCar/BMW.urdf.xacro (robot description, xacro)
@@ -1,198 +1,5 @@
 <?xml version="1.0"?>
- <robot name="BMW_Car" xmlns:xacro="http://www.ros.org/wiki/xacro">
-    <xacro:include filename="inertial_macros.xacro"/>
-    <material name="blue">
-        <color rgba="0 0.2 0.9 1"/>
-    </material>
-    <material name="gray">
-        <color rgba="0.1 0.1 0.1 1"/>
-    </material>
-    <material name="darkBlue">
-        <color rgba="0 0 0.1 1"/>
-    </material>
-    <link name="dummy_link"/>
-    <!-- Chassis -->
-    <link name="chassis">
-        <visual>
-            <geometry>
-                <box size="0.6 0.7 0.1"/>
-            </geometry>
-            <origin rpy="0 0 0" xyz="0 0 0"/>
-            <material name="darkBlue"/>
-        </visual>
-        <collision>
-            <geometry>
-                <box size="0.6 0.7 0.1"/>
-            </geometry>
-            <origin rpy="0 0 0" xyz="0 0 0"/>
-        </collision>
-        <xacro:inertial_box mass="0.5" x="0.6" y="0.7" z="0.1">
-            <origin rpy="0 0 0" xyz="0 0 0"/>
-        </xacro:inertial_box>
-    </link>
-    <joint name="chassis_joint" type="fixed">
-        <parent link="dummy_link"/>
-        <child link="chassis"/>
-        <origin xyz="0 0 0"/>
-    </joint>
-    <gazebo reference="chassis">
-        <material>Gazebo/DarkMagentaTransparent</material>
-    </gazebo>
-    <!-- Front Left Wheel -->
-    <link name="LF_wheel">
-        <visual>
-            <geometry>
-                <cylinder radius="0.2" length="0.07"/>
-            </geometry>
-            <material name="gray"/>
-        </visual>
-        <collision>
-            <geometry>
-                <cylinder radius="0.2" length="0.07"/>
-            </geometry>
-        </collision>
-        <xacro:inertial_cylinder mass="0.1" length="0.07" radius="0.2">
-            <origin xyz="0 0 0" rpy="0 0 0"/>
-        </xacro:inertial_cylinder>
-    </link>
-    <joint name="LF_wheel_joint" type="continuous">
-        <parent link="chassis"/>
-        <child link="LF_wheel"/>
-        <origin rpy="0 1.57 0" xyz="-0.333 0.3 0"/>
-        <axis xyz="0 0 -1"/>
-    </joint>
-    <gazebo reference="LF_wheel">
-        <material>Gazebo/Gray</material>
-    </gazebo>
-    <!-- Back Left wheel -->
-    <link name="LB_wheel">
-        <visual>
-            <geometry>
-                <cylinder radius="0.2" length="0.07"/>
-            </geometry>
-            <material name="gray"/>
-        </visual>
-        <collision>
-            <geometry>
-                <cylinder radius="0.2" length="0.07"/>
-            </geometry>
-        </collision>
-        <xacro:inertial_cylinder mass="0.1" length="0.07" radius="0.2">
-            <origin xyz="0 0 0" rpy="0 0 0"/>
-        </xacro:inertial_cylinder>
-    </link>
-    <joint name="LB_wheel_joint" type="continuous">
-        <parent link="chassis"/>
-        <child link="LB_wheel"/>
-        <origin rpy="0 1.57 0" xyz="-0.333 -0.3 0"/>
-        <axis xyz="0 0 -1"/>
-    </joint>
-    <gazebo reference="LB_wheel">
-        <material>Gazebo/Gray</material>
-    </gazebo>
-    <!-- Front Right Wheel -->
-    <link name="RF_wheel">
-        <visual>
-            <geometry>
-                <cylinder radius="0.2" length="0.07"/>
-            </geometry>
-            <material name="gray"/>
-        </visual>
-        <collision>
-            <geometry>
-                <cylinder radius="0.2" length="0.07"/>
-            </geometry>
-        </collision>
-        <xacro:inertial_cylinder mass="0.1" length="0.07" radius="0.2">
-            <origin xyz="0 0 0" rpy="0 0 0"/>
-        </xacro:inertial_cylinder>
-    </link>
-    <joint name="RF_wheel_joint" type="continuous">
-        <parent link="chassis"/>
-        <child link="RF_wheel"/>
-        <origin rpy="0 1.57 0" xyz="0.333 0.3 0"/>
-        <axis xyz="0 0 1"/>
-    </joint>
-    <gazebo reference="RF_wheel">
-        <material>Gazebo/Gray</material>
-    </gazebo>
-    <!-- Back Right Wheel -->
-    <link name="RB_wheel">
-        <visual>
-            <geometry>
-                <cylinder radius="0.2" length="0.07"/>
-            </geometry>
-            <material name="gray"/>
-        </visual>
-        <collision>
-            <geometry>
-                <cylinder radius="0.2" length="0.07"/>
-            </geometry>
-        </collision>
-        <xacro:inertial_cylinder mass="0.1" length="0.07" radius="0.2">
-            <origin xyz="0 0 0" rpy="0 0 0"/>
-        </xacro:inertial_cylinder>
-    </link>
-    <joint name="RB_wheel_joint" type="continuous">
-        <parent link="chassis"/>
-        <child link="RB_wheel"/>
-        <origin rpy="0 1.57 0" xyz="0.333 -0.3 0"/>
-        <axis xyz="0 0 1"/>
-    </joint>
-    <gazebo reference="RB_wheel">
-        <material>Gazebo/Gray</material>
-    </gazebo>
-    <!-- Lidar -->
-    <link name="lidar">
-        <visual>
-            <geometry>
-                <cylinder radius="0.15" length="0.25"/>
-            </geometry>
-            <origin rpy="0 0 0" xyz="0 -0.16 0.1"/>
-            <material name="blue"/>
-        </visual>
-        <collision>
-            <geometry>
-                <cylinder radius="0.15" length="0.25"/>
-            </geometry>
-        </collision>
-        <xacro:inertial_cylinder mass="0.2" length="0.25" radius="0.15">
-            <origin xyz="0 0 0" rpy="0 0 0"/>
-        </xacro:inertial_cylinder>
-    </link>
-    <joint name="lidar_joint" type="fixed">
-        <parent link="chassis"/>
-        <child link="lidar"/>
-        <origin rpy="0 0 0" xyz="0 0 0"/>
-    </joint>
-    <gazebo reference="lidar">
-        <material>Gazebo/Indigo</material>
-    </gazebo>
-    <!-- Camera-->
-    <link name="camera">
-        <visual>
-            <geometry>
-                <box size="0.15 0.15 0.08"/>
-            </geometry>
-            <origin rpy="0 0 0" xyz="0 0.2 0.05"/>
-            <material name="blue"/>
-        </visual>
-        <collision>
-            <geometry>
-                <box size="0.15 0.15 0.08"/>
-            </geometry>
-            <origin rpy="0 0 0" xyz="0 0.2 0.05"/>
-        </collision>
-        <xacro:inertial_box mass="0.2" x="0.15" y="0.15" z="0.08">
-            <origin rpy="0 0 0" xyz="0 0 0"/>
-        </xacro:inertial_box>
-    </link>
-    <joint name="camera_joint" type="fixed">
-        <parent link="chassis"/>
-        <child link="camera"/>
-        <origin rpy="0 0 0" xyz="0 0 0"/>
-    </joint>
-    <gazebo reference="camera">
-        <material>Gazebo/Indigo</material>
-    </gazebo>
- </robot>
+<robot name="BMW_Car" xmlns:xacro="http://www.ros.org/wiki/xacro">
+  <xacro:include filename="BMW_core.xacro"/>
+  <xacro:include filename="gazebo_control.xacro"/>
+</robot>
