Commit message: added gazebo materials

File: src/robot_description/models/myCar/BMW.urdf (robot description, URDF)
Before this commit: robot BMW_Car, 8 links, 7 joints
Links:
- removed link world
- added link dummy_link
- link LB_wheel: mass None -> 0.1
- link LF_wheel: mass None -> 0.1
- link RB_wheel: mass None -> 0.1
- link RF_wheel: mass None -> 0.1
- link camera: mass None -> 0.2
- link chassis: mass None -> 0.5
- link lidar: mass None -> 0.2
Joints:
- joint chassis_joint: parent world -> dummy_link

Commit message: added camera sensor

File: src/robot_description/models/myCar/BMW.urdf (robot description, URDF)
Before this commit: robot BMW_Car, 8 links, 7 joints
Joints:
- joint RB_wheel_joint: axis 0 0 1 -> 0 0 -1
- joint RF_wheel_joint: axis 0 0 1 -> 0 0 -1

File: src/robot_description/models/myCar/BMW.urdf.xacro (robot description, xacro)
@@ -4,3 +4,4 @@
   <xacro:include filename="gazebo_control.xacro"/>
   <xacro:include filename="lidar.xacro"/>
+  <xacro:include filename="camera.xacro"/>
 </robot>

Commit message: change urdf model so that x axis is in the forward direction

File: src/robot_description/models/myCar/BMW.urdf (robot description, URDF)
Before this commit: robot BMW_Car, 8 links, 7 joints
Joints:
- joint LB_wheel_joint: origin xyz=-0.333 -0.3 0 rpy=0 1.57 0 -> xyz=-0.333 -0.333 0 rpy=0 1.57 -1.57
- joint LF_wheel_joint: origin xyz=-0.333 0.3 0 rpy=0 1.57 0 -> xyz=-0.333 0.333 0 rpy=0 1.57 -1.57
- joint RB_wheel_joint: origin xyz=0.333 -0.3 0 rpy=0 1.57 0 -> xyz=0.333 -0.333 0 rpy=0 1.57 -1.57
- joint RF_wheel_joint: origin xyz=0.333 0.3 0 rpy=0 1.57 0 -> xyz=0.333 0.333 0 rpy=0 1.57 -1.57

File: src/robot_description/models/myCar/BMW_core.xacro (robot description, xacro)
@@ -18,5 +18,5 @@
                 <box size="0.6 0.7 0.1"/>
             </geometry>
-            <origin rpy="0 0 0" xyz="0 0 0"/>
+            <origin rpy="0 0 1.57" xyz="0 0 0"/>
             <material name="darkBlue"/>
         </visual>
@@ -25,8 +25,8 @@
                 <box size="0.6 0.7 0.1"/>
             </geometry>
-            <origin rpy="0 0 0" xyz="0 0 0"/>
+            <origin rpy="0 0 1.57" xyz="0 0 0"/>
         </collision>
         <xacro:inertial_box mass="0.5" x="0.6" y="0.7" z="0.1">
-            <origin rpy="0 0 0" xyz="0 0 0"/>
+            <origin rpy="0 0 1.57" xyz="0 0 0"/>
         </xacro:inertial_box>
     </link>
@@ -59,5 +59,5 @@
         <parent link="chassis"/>
         <child link="LF_wheel"/>
-        <origin rpy="0 1.57 0" xyz="-0.333 0.3 0"/>
+        <origin rpy="0 1.57 -1.57" xyz="-0.333 0.333 0"/>
         <axis xyz="0 0 -1"/>
     </joint>
@@ -85,5 +85,5 @@
         <parent link="chassis"/>
         <child link="LB_wheel"/>
-        <origin rpy="0 1.57 0" xyz="-0.333 -0.3 0"/>
+        <origin rpy="0 1.57 -1.57" xyz="-0.333 -0.333 0"/>
         <axis xyz="0 0 -1"/>
     </joint>
@@ -111,5 +111,5 @@
         <parent link="chassis"/>
         <child link="RF_wheel"/>
-        <origin rpy="0 1.57 0" xyz="0.333 0.3 0"/>
+        <origin rpy="0 1.57 -1.57" xyz="0.333 0.333 0"/>
         <axis xyz="0 0 -1"/>
     </joint>
@@ -137,5 +137,5 @@
         <parent link="chassis"/>
         <child link="RB_wheel"/>
-        <origin rpy="0 1.57 0" xyz="0.333 -0.3 0"/>
+        <origin rpy="0 1.57 -1.57" xyz="0.333 -0.333 0"/>
         <axis xyz="0 0 -1"/>
     </joint>
@@ -149,5 +149,5 @@
                 <cylinder radius="0.15" length="0.25"/>
             </geometry>
-            <origin rpy="0 0 0" xyz="0 -0.16 0.1"/>
+            <origin rpy="0 0 0" xyz="-0.16 0 0.1"/>
             <material name="blue"/>
         </visual>
@@ -158,5 +158,5 @@
         </collision>
         <xacro:inertial_cylinder mass="0.2" length="0.25" radius="0.15">
-            <origin xyz="0 0 0" rpy="0 0 0"/>
+            <origin rpy="0 0 0" xyz="-0.16 0 0.1"/>
         </xacro:inertial_cylinder>
     </link>
@@ -175,5 +175,5 @@
                 <box size="0.15 0.15 0.08"/>
             </geometry>
-            <origin rpy="0 0 0" xyz="0 0.2 0.05"/>
+            <origin rpy="0 0 0" xyz="0.2 0 0.05"/>
             <material name="blue"/>
         </visual>
@@ -182,5 +182,5 @@
                 <box size="0.15 0.15 0.08"/>
             </geometry>
-            <origin rpy="0 0 0" xyz="0 0.2 0.05"/>
+            <origin rpy="0 0 0" xyz="0.2 0 0.05"/>
         </collision>
         <xacro:inertial_box mass="0.2" x="0.15" y="0.15" z="0.08">

File: src/robot_description/models/myCar/camera.xacro (robot description, xacro)
@@ -5,5 +5,5 @@
       <update_rate>10.0</update_rate>
       <camera name="camera1">
-        <pose>0 -0.15 0 0 0 -1.57</pose>
+        <pose>0 0.3 0 0 0 1.57</pose>
         <horizontal_fov>1.4</horizontal_fov>
         <image>

Commit message: updated pysical properties of the robot

File: src/robot_description/models/myCar/BMW.urdf (robot description, URDF)
Before this commit: robot BMW_Car, 8 links, 7 joints
Links:
- link LB_wheel: mass 0.1 -> 0.05; geometry collision sphere radius=0.2; visual cylinder length=0.07 radius=0.2
- link LF_wheel: mass 0.1 -> 0.05; geometry collision sphere radius=0.2; visual cylinder length=0.07 radius=0.2
- link RB_wheel: mass 0.1 -> 0.05; geometry collision sphere radius=0.2; visual cylinder length=0.07 radius=0.2
- link RF_wheel: mass 0.1 -> 0.05; geometry collision sphere radius=0.2; visual cylinder length=0.07 radius=0.2
- link camera: mass 0.2 -> 0.05
- link chassis: mass 0.5 -> 0.1
- link lidar: mass 0.2 -> 0.1
Joints:
- joint LB_wheel_joint: origin xyz=-0.333 -0.333 0 rpy=0 1.57 -1.57 -> xyz=-0.333 0.333 0 rpy=0 1.57 -1.57
- joint LF_wheel_joint: origin xyz=-0.333 0.333 0 rpy=0 1.57 -1.57 -> xyz=0.333 0.333 0 rpy=0 1.57 -1.57
- joint RB_wheel_joint: origin xyz=0.333 -0.333 0 rpy=0 1.57 -1.57 -> xyz=-0.333 -0.333 0 rpy=0 1.57 -1.57
- joint RF_wheel_joint: origin xyz=0.333 0.333 0 rpy=0 1.57 -1.57 -> xyz=0.333 -0.333 0 rpy=0 1.57 -1.57

File: src/robot_description/models/myCar/BMW.urdf.xacro (robot description, xacro)
@@ -2,6 +2,6 @@
 <robot name="BMW_Car" xmlns:xacro="http://www.ros.org/wiki/xacro">
   <xacro:include filename="BMW_core.xacro"/>
-  <!-- <xacro:include filename="gazebo_cont rol.xacro"/> -->
-  <xacro:include filename="ros2_control.xacro"/>
+  <xacro:include filename="gazebo_control.xacro"/>
+  <!-- <xacro:include filename="ros2_control.xacro"/> -->
   <xacro:include filename="lidar.xacro"/>
   <xacro:include filename="camera.xacro"/>

File: src/robot_description/models/myCar/BMW_core.xacro (robot description, xacro)
@@ -2,4 +2,5 @@
  <robot xmlns:xacro="http://www.ros.org/wiki/xacro">
     <xacro:include filename="inertial_macros.xacro"/>
+    <xacro:property name="wheel_mass" value="0.05"/>
     <material name="blue">
         <color rgba="0 0.2 0.9 1"/>
@@ -27,5 +28,5 @@
             <origin rpy="0 0 1.57" xyz="0 0 0"/>
         </collision>
-        <xacro:inertial_box mass="0.5" x="0.6" y="0.7" z="0.1">
+        <xacro:inertial_box mass="0.1" x="0.6" y="0.7" z="0.1">
             <origin rpy="0 0 1.57" xyz="0 0 0"/>
         </xacro:inertial_box>
@@ -40,4 +41,60 @@
     </gazebo>
     <!-- Front Left Wheel -->
+    <link name="LB_wheel">
+        <visual>
+            <geometry>
+                <cylinder radius="0.2" length="0.07"/>
+            </geometry>
+            <material name="gray"/>
+        </visual>
+        <collision>
+            <geometry>
+                <sphere radius="0.2"/>
+            </geometry>
+        </collision>
+        <xacro:inertial_cylinder mass="${wheel_mass}" length="0.07" radius="0.2">
+            <origin xyz="0 0 0" rpy="0 0 0"/>
+        </xacro:inertial_cylinder>
+    </link>
+    <joint name="LB_wheel_joint" type="continuous">
+        <parent link="chassis"/>
+        <child link="LB_wheel"/>
+        <origin rpy="0 1.57 -1.57" xyz="-0.333 0.333 0"/>
+        <axis xyz="0 0 -1"/>
+    </joint>
+    <gazebo reference="LB_wheel">
+        <material>Gazebo/Gray</material>
+        <mu1 value="0.2"/>
+        <mu2 value="0.2"/>
+    </gazebo>
+    <!-- Back Left wheel -->
+    <link name="RB_wheel">
+        <visual>
+            <geometry>
+                <cylinder radius="0.2" length="0.07"/>
+            </geometry>
+            <material name="gray"/>
+        </visual>
+        <collision>
+            <geometry>
+                <sphere radius="0.2"/>
+            </geometry>
+        </collision>
+        <xacro:inertial_cylinder mass="${wheel_mass}" length="0.07" radius="0.2">
+            <origin xyz="0 0 0" rpy="0 0 0"/>
+        </xacro:inertial_cylinder>
+    </link>
+    <joint name="RB_wheel_joint" type="continuous">
+        <parent link="chassis"/>
+        <child link="RB_wheel"/>
+        <origin rpy="0 1.57 -1.57" xyz="-0.333 -0.333 0"/>
+        <axis xyz="0 0 -1"/>
+    </joint>
+    <gazebo reference="RB_wheel">
+        <material>Gazebo/Gray</material>
+        <mu1 value="0.2"/>
+        <mu2 value="0.2"/>
+    </gazebo>
+    <!-- Front Right Wheel -->
     <link name="LF_wheel">
         <visual>
@@ -49,8 +106,8 @@
         <collision>
             <geometry>
-                <cylinder radius="0.2" length="0.07"/>
-            </geometry>
-        </collision>
-        <xacro:inertial_cylinder mass="0.1" length="0.07" radius="0.2">
+                <sphere radius="0.2"/>
+            </geometry>
+        </collision>
+        <xacro:inertial_cylinder mass="${wheel_mass}" length="0.07" radius="0.2">
             <origin xyz="0 0 0" rpy="0 0 0"/>
         </xacro:inertial_cylinder>
@@ -59,37 +116,13 @@
         <parent link="chassis"/>
         <child link="LF_wheel"/>
-        <origin rpy="0 1.57 -1.57" xyz="-0.333 0.333 0"/>
+        <origin rpy="0 1.57 -1.57" xyz="0.333 0.333 0"/>
         <axis xyz="0 0 -1"/>
     </joint>
     <gazebo reference="LF_wheel">
         <material>Gazebo/Gray</material>
-    </gazebo>
-    <!-- Back Left wheel -->
-    <link name="LB_wheel">
-        <visual>
-            <geometry>
-                <cylinder radius="0.2" length="0.07"/>
-            </geometry>
-            <material name="gray"/>
-        </visual>
-        <collision>
-            <geometry>
-                <cylinder radius="0.2" length="0.07"/>
-            </geometry>
-        </collision>
-        <xacro:inertial_cylinder mass="0.1" length="0.07" radius="0.2">
-            <origin xyz="0 0 0" rpy="0 0 0"/>
-        </xacro:inertial_cylinder>
-    </link>
-    <joint name="LB_wheel_joint" type="continuous">
-        <parent link="chassis"/>
-        <child link="LB_wheel"/>
-        <origin rpy="0 1.57 -1.57" xyz="-0.333 -0.333 0"/>
-        <axis xyz="0 0 -1"/>
-    </joint>
-    <gazebo reference="LB_wheel">
-        <material>Gazebo/Gray</material>
-    </gazebo>
-    <!-- Front Right Wheel -->
+        <mu1 value="0.2"/>
+        <mu2 value="0.2"/>
+    </gazebo>
+    <!-- Back Right Wheel -->
     <link name="RF_wheel">
         <visual>
@@ -101,8 +134,8 @@
         <collision>
             <geometry>
-                <cylinder radius="0.2" length="0.07"/>
-            </geometry>
-        </collision>
-        <xacro:inertial_cylinder mass="0.1" length="0.07" radius="0.2">
+                <sphere radius="0.2"/>
+            </geometry>
+        </collision>
+        <xacro:inertial_cylinder mass="${wheel_mass}" length="0.07" radius="0.2">
             <origin xyz="0 0 0" rpy="0 0 0"/>
         </xacro:inertial_cylinder>
@@ -111,35 +144,11 @@
         <parent link="chassis"/>
         <child link="RF_wheel"/>
-        <origin rpy="0 1.57 -1.57" xyz="0.333 0.333 0"/>
+        <origin rpy="0 1.57 -1.57" xyz="0.333 -0.333 0"/>
         <axis xyz="0 0 -1"/>
     </joint>
     <gazebo reference="RF_wheel">
         <material>Gazebo/Gray</material>
-    </gazebo>
-    <!-- Back Right Wheel -->
-    <link name="RB_wheel">
-        <visual>
-            <geometry>
-                <cylinder radius="0.2" length="0.07"/>
-            </geometry>
-            <material name="gray"/>
-        </visual>
-        <collision>
-            <geometry>
-                <cylinder radius="0.2" length="0.07"/>
-            </geometry>
-        </collision>
-        <xacro:inertial_cylinder mass="0.1" length="0.07" radius="0.2">
-            <origin xyz="0 0 0" rpy="0 0 0"/>
-        </xacro:inertial_cylinder>
-    </link>
-    <joint name="RB_wheel_joint" type="continuous">
-        <parent link="chassis"/>
-        <child link="RB_wheel"/>
-        <origin rpy="0 1.57 -1.57" xyz="0.333 -0.333 0"/>
-        <axis xyz="0 0 -1"/>
-    </joint>
-    <gazebo reference="RB_wheel">
-        <material>Gazebo/Gray</material>
+        <mu1 value="0.2"/>
+        <mu2 value="0.2"/>
     </gazebo>
     <!-- Lidar -->
@@ -156,6 +165,7 @@
                 <cylinder radius="0.15" length="0.25"/>
             </geometry>
-        </collision>
-        <xacro:inertial_cylinder mass="0.2" length="0.25" radius="0.15">
+            <origin rpy="0 0 0" xyz="-0.16 0 0.1"/>
+        </collision>
+        <xacro:inertial_cylinder mass="0.1" length="0.25" radius="0.15">
             <origin rpy="0 0 0" xyz="-0.16 0 0.1"/>
         </xacro:inertial_cylinder>
@@ -184,5 +194,5 @@
             <origin rpy="0 0 0" xyz="0.2 0 0.05"/>
         </collision>
-        <xacro:inertial_box mass="0.2" x="0.15" y="0.15" z="0.08">
+        <xacro:inertial_box mass="0.05" x="0.15" y="0.15" z="0.08">
             <origin rpy="0 0 0" xyz="0 0 0"/>
         </xacro:inertial_box>

File: src/robot_description/models/myCar/camera.xacro (robot description, xacro)
@@ -5,5 +5,5 @@
       <update_rate>10.0</update_rate>
       <camera name="camera1">
-        <pose>0 0.3 0 0 0 1.57</pose>
+        <pose>1 0 0 0 0 0</pose>
         <horizontal_fov>1.4</horizontal_fov>
         <image>
