Commit message: fixed rotation axis

File: src/robot_description/models/myCar/BMW_core.xacro (robot description, xacro)
@@ -112,5 +112,5 @@
         <child link="RF_wheel"/>
         <origin rpy="0 1.57 0" xyz="0.333 0.3 0"/>
-        <axis xyz="0 0 1"/>
+        <axis xyz="0 0 -1"/>
     </joint>
     <gazebo reference="RF_wheel">
@@ -138,5 +138,5 @@
         <child link="RB_wheel"/>
         <origin rpy="0 1.57 0" xyz="0.333 -0.3 0"/>
-        <axis xyz="0 0 1"/>
+        <axis xyz="0 0 -1"/>
     </joint>
     <gazebo reference="RB_wheel">

Commit message: update world and robot

File: src/robot_description/models/myCar/BMW_core.xacro (robot description, xacro)
@@ -64,5 +64,5 @@
     </joint>
     <gazebo reference="LB_wheel">
-        <material>Gazebo/Gray</material>
+        <material>Gazebo/Black</material>
         <mu1 value="0.2"/>
         <mu2 value="0.2"/>
@@ -92,5 +92,5 @@
     </joint>
     <gazebo reference="RB_wheel">
-        <material>Gazebo/Gray</material>
+        <material>Gazebo/Black</material>
         <mu1 value="0.2"/>
         <mu2 value="0.2"/>
@@ -120,5 +120,5 @@
     </joint>
     <gazebo reference="LF_wheel">
-        <material>Gazebo/Gray</material>
+        <material>Gazebo/Black</material>
         <mu1 value="0.2"/>
         <mu2 value="0.2"/>
@@ -148,5 +148,5 @@
     </joint>
     <gazebo reference="RF_wheel">
-        <material>Gazebo/Gray</material>
+        <material>Gazebo/Black</material>
         <mu1 value="0.2"/>
         <mu2 value="0.2"/>
